Commit message: Modified pr100_ws remote_ws the robot wheel/caster location.

File: pr100_ws/src/pr100_description/urdf/macros.xacro (robot description, xacro)
@@ -44,27 +44,28 @@
         </link>
         <gazebo reference="${lr}_wheel">
-        <mu1 value="1.0"/>
-        <mu2 value="1.0"/>
-        <kp  value="10000000.0" />
-        <kd  value="1.0" />
-        <fdir1 value="1 0 0"/>
-        <material>Gazebo/Black</material>
+            <mu1 value="1.0"/>
+            <mu2 value="1.0"/>
+            <kp  value="10000000.0" />
+            <kd  value="1.0" />
+            <fdir1 value="1 0 0"/>
+            <material>Gazebo/Black</material>
         </gazebo>
         <joint name="${lr}_wheel_hinge" type="continuous">
-        <parent link="chassis"/>
-        <child link="${lr}_wheel"/>
-        <origin xyz="${chassisLength/3} ${tY*wheelWidth/2+tY*chassisWidth/2} ${casterRadius+2*wheelRadius-chassisHeight}" rpy="0 0 0" />
-        <!-- <origin xyz="${-wheelPos+chassisLength/2} ${tY*wheelWidth/2+tY*chassisWidth/2} ${wheelRadius}" rpy="0 0 0" /> -->
-        <axis xyz="0 1 0" rpy="0 0 0" />
-        <limit effort="100" velocity="100"/>
-        <joint_properties damping="0.0" friction="0.0"/>
+            <parent link="chassis"/>
+            <child link="${lr}_wheel"/>
+            <origin xyz="0.05 ${tY*wheelWidth/2+tY*chassisWidth/2} ${casterRadius+2*wheelRadius-chassisHeight}" rpy="0 0 0" />
+            <!-- <origin xyz="${chassisLength/3} ${tY*wheelWidth/2+tY*chassisWidth/2} ${casterRadius+2*wheelRadius-chassisHeight}" rpy="0 0 0" /> -->
+            <!-- <origin xyz="${-wheelPos+chassisLength/2} ${tY*wheelWidth/2+tY*chassisWidth/2} ${wheelRadius}" rpy="0 0 0" /> -->
+            <axis xyz="0 1 0" rpy="0 0 0" />
+            <limit effort="100" velocity="100"/>
+            <joint_properties damping="0.0" friction="0.0"/>
         </joint>
         <transmission name="${lr}_trans">
-        <type>transmission_interface/SimpleTransmission</type>
-        <joint name="${lr}_wheel_hinge"/>
-        <actuator name="${lr}Motor">
-            <hardwareInterface>EffortJointInterface</hardwareInterface>
-            <mechanicalReduction>10</mechanicalReduction>
-        </actuator>
+            <type>transmission_interface/SimpleTransmission</type>
+            <joint name="${lr}_wheel_hinge"/>
+            <actuator name="${lr}Motor">
+                <hardwareInterface>EffortJointInterface</hardwareInterface>
+                <mechanicalReduction>10</mechanicalReduction>
+            </actuator>
         </transmission>
     </xacro:macro>

File: pr100_ws/src/pr100_description/urdf/pr100.xacro (robot description, xacro)
@@ -9,5 +9,5 @@
     <xacro:property name="chassisMass" value="50"/>
     <xacro:property name="casterRadius" value="0.05"/>
-    <xacro:property name="casterMass" value="5"/>
+    <xacro:property name="casterMass" value="1"/>
     <!-- 0.05*0.1*0.5 * 5 -->
     <xacro:property name="wheelWidth" value="0.01"/>
@@ -55,5 +55,6 @@
     <link name="caster_wheel">
         <collision>
-            <origin xyz="${casterRadius-chassisLength/2} 0 ${casterRadius-chassisHeight+2*wheelRadius}" rpy="0 0 0"/>
+            <origin xyz="${-casterRadius} 0 ${casterRadius-chassisHeight+2*wheelRadius}" rpy="0 0 0"/>
+            <!-- <origin xyz="${casterRadius-chassisLength/2} 0 ${casterRadius-chassisHeight+2*wheelRadius}" rpy="0 0 0"/> -->
             <geometry>
             <sphere radius="${casterRadius}"/>
@@ -61,5 +62,6 @@
         </collision>
         <visual>
-            <origin xyz="${casterRadius-chassisLength/2} 0 ${casterRadius-chassisHeight+2*wheelRadius}" rpy="0 0 0"/>
+            <origin xyz="${-casterRadius} 0 ${casterRadius-chassisHeight+2*wheelRadius}" rpy="0 0 0"/>
+            <!-- <origin xyz="${casterRadius-chassisLength/2} 0 ${casterRadius-chassisHeight+2*wheelRadius}" rpy="0 0 0"/> -->
             <geometry>
             <sphere radius="${casterRadius}"/>
@@ -68,13 +70,39 @@
         </visual>
         <inertial>
-            <origin xyz="${casterRadius-chassisLength/2} 0 ${casterRadius-chassisHeight+2*wheelRadius}" rpy="0 0 0"/>
+            <origin xyz="${-casterRadius} 0 ${casterRadius-chassisHeight+2*wheelRadius}" rpy="0 0 0"/>
+            <!-- <origin xyz="${casterRadius-chassisLength/2} 0 ${casterRadius-chassisHeight+2*wheelRadius}" rpy="0 0 0"/> -->
             <mass value="${casterMass}"/>
             <xacro:sphere_inertia m="${casterMass}" r="${casterRadius}"/>
         </inertial>
     </link>
-    <joint name="fixed" type="fixed">
+    <joint name="fixed_caster_joint" type="fixed">
         <parent link="chassis"/>
         <child link="caster_wheel"/>
     </joint>
+    <!-- caster_wheel 2 -->
+    <!-- <link name="caster_wheel2">
+        <collision>
+            <origin xyz="${chassisLength/2-casterRadius} 0 ${casterRadius-chassisHeight+2*wheelRadius}" rpy="0 0 0"/>
+            <geometry>
+            <sphere radius="${casterRadius}"/>
+            </geometry>
+        </collision>
+        <visual>
+            <origin xyz="${chassisLength/2-casterRadius} 0 ${casterRadius-chassisHeight+2*wheelRadius}" rpy="0 0 0"/>
+            <geometry>
+            <sphere radius="${casterRadius}"/>
+            </geometry>
+            <material name="black"/>
+        </visual>
+        <inertial>
+            <origin xyz="${chassisLength/2-casterRadius} 0 ${casterRadius-chassisHeight+2*wheelRadius}" rpy="0 0 0"/>
+            <mass value="${casterMass}"/>
+            <xacro:sphere_inertia m="${casterMass}" r="${casterRadius}"/>
+        </inertial>
+    </link>
+    <joint name="fixed_caster_joint2" type="fixed">
+        <parent link="chassis"/>
+        <child link="caster_wheel2"/>
+    </joint> -->
     <!-- right wheel link -->
     <!-- right wheel joint -->
