Commit message: pr100_ws Saving progress...

File: pr100_ws/src/pr100_description/urdf/pr100.xacro (robot description, xacro)
@@ -17,4 +17,5 @@
     <xacro:property name="cameraSize" value="0.05"/>
     <xacro:property name="cameraMass" value="0.1"/>
+    <xacro:property name="sonarSize" value="0.1"/>
     <!-- include files -->
     <xacro:include filename="$(find pr100_description)/urdf/pr100.gazebo" />
@@ -110,3 +111,31 @@
         <child link="hokuyo"/>
     </joint>
+    <!-- Camera -->
+    <link name="camera">
+        <collision>
+        <origin xyz="0 0 0" rpy="0 0 0"/>
+        <geometry>
+            <box size="${cameraSize} ${cameraSize} ${cameraSize}"/>
+        </geometry>
+        </collision>
+        <visual>
+        <origin xyz="0 0 0" rpy="0 0 0"/>
+        <geometry>
+            <box size="${cameraSize} ${cameraSize} ${cameraSize}"/>
+        </geometry>
+        <material name="green"/>
+        </visual>
+        <inertial>
+        <mass value="${cameraMass}" />
+        <origin xyz="0 0 0" rpy="0 0 0"/>
+        <box_inertia m="${cameraMass}" x="${cameraSize}" y="${cameraSize}" z="${cameraSize}" />
+        <inertia ixx="1e-6" ixy="0" ixz="0" iyy="1e-6" iyz="0" izz="1e-6" />
+        </inertial>
+    </link>
+    <joint name="camera_joint" type="fixed">
+        <axis xyz="0 1 0" />
+        <origin xyz="${chassisWidth/2} 0 0" rpy="0 0 0"/>
+        <parent link="chassis"/>
+        <child link="camera"/>
+    </joint>
 </robot>

Commit message: Put ultrasonic sensor on pr100

File: pr100_ws/src/pr100_description/urdf/pr100.xacro (robot description, xacro)
@@ -84,51 +84,78 @@
     <xacro:wheel lr="left" tY="0.5"/>
     <!-- sensor -->
-    <!-- Hokuyo Laser -->
-    <link name="hokuyo">
+    <!-- sonar (ultrasonic) -->
+    <link name="sonar1">
         <collision>
-        <origin xyz="0 0 0" rpy="0 0 0"/>
-        <geometry>
-        <box size="0.1 0.1 0.1"/>
-        </geometry>
+            <origin xyz="0 0 0" rpy="0 0 0"/>
+            <geometry>
+                <box size="0.01 0.01 0.01"/>
+            </geometry>
         </collision>
         <visual>
-        <origin xyz="0 0 0" rpy="0 0 0"/>
-        <geometry>
-            <mesh filename="package://pr100_description/meshes/hokuyo.dae"/>
-        </geometry>
+            <origin xyz="0 0 0" rpy="0 0 0"/>
+            <geometry>
+                <box size="0.01 0.01 0.01"/>
+            </geometry>
+            <material name="black"/>
         </visual>
         <inertial>
-        <mass value="1e-5" />
-        <origin xyz="0 0 0" rpy="0 0 0"/>
-        <inertia ixx="1e-6" ixy="0" ixz="0" iyy="1e-6" iyz="0" izz="1e-6" />
+            <mass value="1e-5" />
+            <origin xyz="0 0 0" rpy="0 0 0"/>
+            <inertia ixx="1e-6" ixy="0" ixz="0" iyy="1e-6" iyz="0" izz="1e-6" />
         </inertial>
     </link>
-    <joint name="hokuyo_joint" type="fixed">
+    <joint name="sonar_joint1" type="fixed">
         <axis xyz="0 1 0" />
-        <!-- <origin xyz=".15 0 .1" rpy="0 0 0"/> -->
-        <origin xyz="0 0 ${chassisHeight/2+chassisHeight*0.01}" rpy="0 0 0"/>
+        <origin xyz="${chassisHeight/2} ${chassisHeight/3} ${chassisHeight/3+chassisHeight*0.01}" rpy="0 0 0"/>
         <parent link="chassis"/>
-        <child link="hokuyo"/>
+        <child link="sonar1"/>
+    </joint>
+    <!-- sonar (ultrasonic) -->
+    <link name="sonar2">
+        <collision>
+            <origin xyz="0 0 0" rpy="0 0 0"/>
+            <geometry>
+                <box size="0.01 0.01 0.01"/>
+            </geometry>
+        </collision>
+        <visual>
+            <origin xyz="0 0 0" rpy="0 0 0"/>
+            <geometry>
+                <box size="0.01 0.01 0.01"/>
+            </geometry>
+            <material name="black"/>
+        </visual>
+        <inertial>
+            <mass value="1e-5" />
+            <origin xyz="0 0 0" rpy="0 0 0"/>
+            <inertia ixx="1e-6" ixy="0" ixz="0" iyy="1e-6" iyz="0" izz="1e-6" />
+        </inertial>
+    </link>
+    <joint name="sonar_joint2" type="fixed">
+        <axis xyz="0 1 0" />
+        <origin xyz="${chassisHeight/2} ${-chassisHeight/3} ${chassisHeight/3+chassisHeight*0.01}" rpy="0 0 0"/>
+        <parent link="chassis"/>
+        <child link="sonar2"/>
     </joint>
     <!-- Camera -->
     <link name="camera">
         <collision>
-        <origin xyz="0 0 0" rpy="0 0 0"/>
-        <geometry>
-            <box size="${cameraSize} ${cameraSize} ${cameraSize}"/>
-        </geometry>
+            <origin xyz="0 0 0" rpy="0 0 0"/>
+            <geometry>
+                <box size="${cameraSize} ${cameraSize} ${cameraSize}"/>
+            </geometry>
         </collision>
         <visual>
-        <origin xyz="0 0 0" rpy="0 0 0"/>
-        <geometry>
-            <box size="${cameraSize} ${cameraSize} ${cameraSize}"/>
-        </geometry>
-        <material name="green"/>
+            <origin xyz="0 0 0" rpy="0 0 0"/>
+            <geometry>
+                <box size="${cameraSize} ${cameraSize} ${cameraSize}"/>
+            </geometry>
+            <material name="green"/>
         </visual>
         <inertial>
-        <mass value="${cameraMass}" />
-        <origin xyz="0 0 0" rpy="0 0 0"/>
-        <box_inertia m="${cameraMass}" x="${cameraSize}" y="${cameraSize}" z="${cameraSize}" />
-        <inertia ixx="1e-6" ixy="0" ixz="0" iyy="1e-6" iyz="0" izz="1e-6" />
+            <mass value="${cameraMass}" />
+            <origin xyz="0 0 0" rpy="0 0 0"/>
+            <box_inertia m="${cameraMass}" x="${cameraSize}" y="${cameraSize}" z="${cameraSize}" />
+            <inertia ixx="1e-6" ixy="0" ixz="0" iyy="1e-6" iyz="0" izz="1e-6" />
         </inertial>
     </link>

Commit message: Update pr100_remote_ws pr100_drive algo decisions.

File: pr100_ws/src/pr100_description/urdf/pr100.xacro (robot description, xacro)
@@ -161,5 +161,6 @@
     </link>
     <joint name="camera_joint" type="fixed">
-        <axis xyz="0 1 0" />
+        <axis xyz="1 0 0" />
+        <!-- <axis xyz="0 1 0" /> -->
         <origin xyz="${chassisWidth/2} 0 0" rpy="0 0 0"/>
         <parent link="chassis"/>

Commit message: In pr100_ws pr100_remote_ws: testing driving algo, added robot models.

File: pr100_ws/src/pr100_description/urdf/pr100.xacro (robot description, xacro)
@@ -9,5 +9,5 @@
     <xacro:property name="chassisMass" value="50"/>
     <xacro:property name="casterRadius" value="0.05"/>
-    <xacro:property name="casterMass" value="1"/>
+    <xacro:property name="casterMass" value="5"/>
     <!-- 0.05*0.1*0.5 * 5 -->
     <xacro:property name="wheelWidth" value="0.01"/>
@@ -28,14 +28,18 @@
         <collision>
             <!-- <origin xyz="0 0 ${wheelRadius}" rpy="0 0 0"/>  -->
-            <origin xyz="0 0 0" rpy="0 0 0"/>
-            <geometry>
-            <box size="${chassisLength} ${chassisWidth} ${chassisHeight}"/>
+            <origin xyz="0 0 -0.15" rpy="0 0 0"/>
+            <!-- <origin xyz="0 0 0" rpy="0 0 0"/>  -->
+            <geometry>
+                <mesh filename="package://pr100_description/meshes/cylinder.stl" scale="0.001 0.001 0.001"/>
+                <!-- <box size="${chassisLength} ${chassisWidth} ${chassisHeight}"/>  -->
             </geometry>
         </collision>
         <visual>
             <!-- <origin xyz="0 0 ${wheelRadius}" rpy="0 0 0"/>  -->
-            <origin xyz="0 0 0" rpy="0 0 0"/>
-            <geometry>
-            <box size="${chassisLength} ${chassisWidth} ${chassisHeight}"/>
+            <origin xyz="0 0 -0.15" rpy="0 0 0"/>
+            <!-- <origin xyz="0 0 0" rpy="0 0 0"/>  -->
+            <geometry>
+                <mesh filename="package://pr100_description/meshes/cylinder.stl" scale="0.001 0.001 0.001"/>
+                <!-- <box size="${chassisLength} ${chassisWidth} ${chassisHeight}"/>  -->
             </geometry>
             <material name="white"/>
@@ -43,5 +47,6 @@
         <inertial>
             <!-- <origin xyz="0 0 ${wheelRadius}" rpy="0 0 0"/>  -->
-            <origin xyz="0 0 0" rpy="0 0 0"/>
+            <origin xyz="0 0 -0.15" rpy="0 0 0"/>
+            <!-- <origin xyz="0 0 0" rpy="0 0 0"/>  -->
             <mass value="${chassisMass}"/>
             <xacro:box_inertia m="${chassisMass}" x="${chassisLength}" y="${chassisWidth}" z="${chassisHeight}"/>
@@ -58,5 +63,5 @@
             <!-- <origin xyz="${casterRadius-chassisLength/2} 0 ${casterRadius-chassisHeight+2*wheelRadius}" rpy="0 0 0"/> -->
             <geometry>
-            <sphere radius="${casterRadius}"/>
+                <sphere radius="${casterRadius}"/>
             </geometry>
         </collision>
@@ -65,5 +70,5 @@
             <!-- <origin xyz="${casterRadius-chassisLength/2} 0 ${casterRadius-chassisHeight+2*wheelRadius}" rpy="0 0 0"/> -->
             <geometry>
-            <sphere radius="${casterRadius}"/>
+                <sphere radius="${casterRadius}"/>
             </geometry>
             <material name="black"/>
